Commit message: Updated mass and inertia values in URDF file

File: my_rb1_description/urdf/my_rb1_robot.urdf (robot description, URDF)
Before this commit: robot robot, 7 links, 6 joints
Links:
- link link_back_caster: mass 1 -> 0.5
- link link_base: mass 10 -> 22
- link link_front_caster: mass 1 -> 0.5
- link link_front_laser: mass 0.5 -> 0

Commit message: Caster wheels replaced to improve movement stability. Torque diminished to increase velocity.

File: my_rb1_description/urdf/my_rb1_robot.urdf (robot description, URDF)
Before this commit: robot robot, 7 links, 6 joints
Joints:
- joint joint_base_back_caster: origin xyz=-0.1 0 -0.15 rpy=0 0 0 -> xyz=-0.2 0 -0.15 rpy=0 0 0
- joint joint_base_front_caster: origin xyz=0.1 0 -0.15 rpy=0 0 0 -> xyz=0.2 0 -0.15 rpy=0 0 0
